File: RF_HAT/RF_HAT_out/CC1200_UHF_432MHz.kicad_sch (KiCad schematic)
At the start: 43 parts, among them J1 SMA, U1 CC1200RHBR, Y1 40MHz

Commit message: switch to SMD pico
Parts:
- TP1, TP2, TP3, TP4: value (none) -> ~

Commit message: switched to 0603 for all passives
Parts:
- C1, C2: footprint Capacitor_SMD:C_0805_2012Metric -> Capacitor_SMD:C_0603_1608Metric; hierarchy_path /03cc9bb1-75ec-4755-9977-259c49401791/0085fed7-e912-48fb-b4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 -> /bd07fb41-9ea7-4d0f-b403-cbcdc979b1cd/31dca4aa-880f-4bf5-8b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; root_uuid 03cc9bb1-75ec-4755-9977-259c49401791 -> bd07fb41-9ea7-4d0f-b403-cbcdc979b1cd
- C10, C11, C12, C13, C14, C15, C16, C17, C3, C4, C5, C6, C7, C8, C9: footprint Capacitor_SMD:C_0402_1005Metric -> Capacitor_SMD:C_0603_1608Metric; hierarchy_path /03cc9bb1-75ec-4755-9977-259c49401791/0085fed7-e912-48fb-b4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 -> /bd07fb41-9ea7-4d0f-b403-cbcdc979b1cd/31dca4aa-880f-4bf5-8b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; root_uuid 03cc9bb1-75ec-4755-9977-259c49401791 -> bd07fb41-9ea7-4d0f-b403-cbcdc979b1cd
- C18, C19, C20, C21, C22, C23, C24, C25, J1, L1, L2, L3, L4, L5, L6, L7, L8, TP1, TP2, TP3, TP4, U1, Y1: hierarchy_path /03cc9bb1-75ec-4755-9977-259c49401791/0085fed7-e912-48fb-b4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 -> /bd07fb41-9ea7-4d0f-b403-cbcdc979b1cd/31dca4aa-880f-4bf5-8b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; root_uuid 03cc9bb1-75ec-4755-9977-259c49401791 -> bd07fb41-9ea7-4d0f-b403-cbcdc979b1cd
- FB1: footprint Inductor_SMD:L_0402_1005Metric -> Inductor_SMD:L_0603_1608Metric; hierarchy_path /03cc9bb1-75ec-4755-9977-259c49401791/0085fed7-e912-48fb-b4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 -> /bd07fb41-9ea7-4d0f-b403-cbcdc979b1cd/31dca4aa-880f-4bf5-8b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; root_uuid 03cc9bb1-75ec-4755-9977-259c49401791 -> bd07fb41-9ea7-4d0f-b403-cbcdc979b1cd
- R1: footprint Resistor_SMD:R_0402_1005Metric -> Resistor_SMD:R_0603_1608Metric; hierarchy_path /03cc9bb1-75ec-4755-9977-259c49401791/0085fed7-e912-48fb-b4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 -> /bd07fb41-9ea7-4d0f-b403-cbcdc979b1cd/31dca4aa-880f-4bf5-8b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; root_uuid 03cc9bb1-75ec-4755-9977-259c49401791 -> bd07fb41-9ea7-4d0f-b403-cbcdc979b1cd
- R2: footprint Resistor_SMD:R_0805_2012Metric -> Resistor_SMD:R_0603_1608Metric; hierarchy_path /03cc9bb1-75ec-4755-9977-259c49401791/0085fed7-e912-48fb-b4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 -> /bd07fb41-9ea7-4d0f-b403-cbcdc979b1cd/31dca4aa-880f-4bf5-8b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; root_uuid 03cc9bb1-75ec-4755-9977-259c49401791 -> bd07fb41-9ea7-4d0f-b403-cbcdc979b1cd

Commit message: first routing of signals
Parts:
- removed TP1, TP2, TP3, TP4: ~, TestPoint:TestPoint_Pad_D1.0mm, symbol Connector:TestPoint
Connections:
- net +3.3V: no longer C10.1, C11.1, C12.1, C13.1, C14.1, C15.1, C16.1, C8.1, C9.1, U1.1 (VDD_GUARD), U1.13 (AVDD_IF), U1.15 (AVDD_RF), U1.22 (AVDD_SYNTH1), U1.25 (AVDD_PFD_CHP), U1.27 (AVDD_SYNTH2), U1.28 (AVDD_XOSC), U1.5 (DVDD)
- net UHF_AVDD_FILT: now also C10.1, C11.1, C12.1, C13.1, C14.1, C15.1, C16.1, C8.1, C9.1, U1.1 (VDD_GUARD), U1.12 (DVDD), U1.13 (AVDD_IF), U1.15 (AVDD_RF), U1.22 (AVDD_SYNTH1), U1.25 (AVDD_PFD_CHP), U1.27 (AVDD_SYNTH2), U1.28 (AVDD_XOSC), U1.5 (DVDD)

Commit message: Restructured kicad schematic for CC1200 PI_HAT readablitity based on M17 reference schematics
Parts:
- removed C11: 47nF, Capacitor_SMD:C_0603_1608Metric, symbol Device:C
- removed C19: 56pF, Capacitor_SMD:C_0603_1608Metric, symbol Device:C
- removed C20: 100pF, Capacitor_SMD:C_0603_1608Metric, symbol Device:C
- removed C22, C25: 5.1pF, Capacitor_SMD:C_0603_1608Metric, symbol Device:C
- removed C23: 6.2pF, Capacitor_SMD:C_0603_1608Metric, symbol Device:C
- removed C24: 2.2pF, Capacitor_SMD:C_0603_1608Metric, symbol Device:C
- removed FB1: 1k@100MHz, Inductor_SMD:L_0603_1608Metric, symbol Device:FerriteBead
- removed R1: 56k, Resistor_SMD:R_0603_1608Metric, symbol Device:R
- removed R2: 18R, Resistor_SMD:R_0603_1608Metric, symbol Device:R
- added C57, C58, C59, C60, C61, C62, C63, C64: 47nF, Capacitor_SMD:C_0603_1608Metric, symbol Device:C
- added R4, R5: 10k, Resistor_SMD:R_0603_1608Metric, symbol Device:R
- added R6: 18R, Resistor_SMD:R_0603_1608Metric, symbol Device:R
- added R7: 56k, Resistor_SMD:R_0603_1608Metric, symbol Device:R
- C1: value 15pF -> 2.2pF; hierarchy_path /bd07fb41-9ea7-4d0f-b403-cbcdc979b1cd/31dca4aa-880f-4bf5-8b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 -> /300cf3d4-e317-44c8-acd8-5f9989779c7c/4304a2bc-ba15-4549-9a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; root_uuid bd07fb41-9ea7-4d0f-b403-cbcdc979b1cd -> 300cf3d4-e317-44c8-acd8-5f9989779c7c
- C10: value 47nF -> 1nF; hierarchy_path /bd07fb41-9ea7-4d0f-b403-cbcdc979b1cd/31dca4aa-880f-4bf5-8b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 -> /300cf3d4-e317-44c8-acd8-5f9989779c7c/4304a2bc-ba15-4549-9a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; root_uuid bd07fb41-9ea7-4d0f-b403-cbcdc979b1cd -> 300cf3d4-e317-44c8-acd8-5f9989779c7c
- C12, C13: value 47nF -> 15pF; hierarchy_path /bd07fb41-9ea7-4d0f-b403-cbcdc979b1cd/31dca4aa-880f-4bf5-8b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 -> /300cf3d4-e317-44c8-acd8-5f9989779c7c/4304a2bc-ba15-4549-9a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; root_uuid bd07fb41-9ea7-4d0f-b403-cbcdc979b1cd -> 300cf3d4-e317-44c8-acd8-5f9989779c7c
- C14, C15, J1, L5, U1, Y1: hierarchy_path /bd07fb41-9ea7-4d0f-b403-cbcdc979b1cd/31dca4aa-880f-4bf5-8b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 -> /300cf3d4-e317-44c8-acd8-5f9989779c7c/4304a2bc-ba15-4549-9a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; root_uuid bd07fb41-9ea7-4d0f-b403-cbcdc979b1cd -> 300cf3d4-e317-44c8-acd8-5f9989779c7c
- C16: value 47nF -> 10nF; hierarchy_path /bd07fb41-9ea7-4d0f-b403-cbcdc979b1cd/31dca4aa-880f-4bf5-8b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 -> /300cf3d4-e317-44c8-acd8-5f9989779c7c/4304a2bc-ba15-4549-9a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; root_uuid bd07fb41-9ea7-4d0f-b403-cbcdc979b1cd -> 300cf3d4-e317-44c8-acd8-5f9989779c7c
- C17: value 10nF -> 220nF; hierarchy_path /bd07fb41-9ea7-4d0f-b403-cbcdc979b1cd/31dca4aa-880f-4bf5-8b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 -> /300cf3d4-e317-44c8-acd8-5f9989779c7c/4304a2bc-ba15-4549-9a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; root_uuid bd07fb41-9ea7-4d0f-b403-cbcdc979b1cd -> 300cf3d4-e317-44c8-acd8-5f9989779c7c
- C18: value 5.1pF -> 1.5nF; hierarchy_path /bd07fb41-9ea7-4d0f-b403-cbcdc979b1cd/31dca4aa-880f-4bf5-8b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 -> /300cf3d4-e317-44c8-acd8-5f9989779c7c/4304a2bc-ba15-4549-9a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; root_uuid bd07fb41-9ea7-4d0f-b403-cbcdc979b1cd -> 300cf3d4-e317-44c8-acd8-5f9989779c7c
- C2: value 15pF -> 39pF; hierarchy_path /bd07fb41-9ea7-4d0f-b403-cbcdc979b1cd/31dca4aa-880f-4bf5-8b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 -> /300cf3d4-e317-44c8-acd8-5f9989779c7c/4304a2bc-ba15-4549-9a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; root_uuid bd07fb41-9ea7-4d0f-b403-cbcdc979b1cd -> 300cf3d4-e317-44c8-acd8-5f9989779c7c
- C21: value 39pF -> 47nF; hierarchy_path /bd07fb41-9ea7-4d0f-b403-cbcdc979b1cd/31dca4aa-880f-4bf5-8b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 -> /300cf3d4-e317-44c8-acd8-5f9989779c7c/4304a2bc-ba15-4549-9a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; root_uuid bd07fb41-9ea7-4d0f-b403-cbcdc979b1cd -> 300cf3d4-e317-44c8-acd8-5f9989779c7c
- C3: value 100nF -> 5.1pF; hierarchy_path /bd07fb41-9ea7-4d0f-b403-cbcdc979b1cd/31dca4aa-880f-4bf5-8b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 -> /300cf3d4-e317-44c8-acd8-5f9989779c7c/4304a2bc-ba15-4549-9a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; root_uuid bd07fb41-9ea7-4d0f-b403-cbcdc979b1cd -> 300cf3d4-e317-44c8-acd8-5f9989779c7c
- C4: value 100nF -> 6.2pF; hierarchy_path /bd07fb41-9ea7-4d0f-b403-cbcdc979b1cd/31dca4aa-880f-4bf5-8b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 -> /300cf3d4-e317-44c8-acd8-5f9989779c7c/4304a2bc-ba15-4549-9a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; root_uuid bd07fb41-9ea7-4d0f-b403-cbcdc979b1cd -> 300cf3d4-e317-44c8-acd8-5f9989779c7c
- C5: value 100nF -> 56pF; hierarchy_path /bd07fb41-9ea7-4d0f-b403-cbcdc979b1cd/31dca4aa-880f-4bf5-8b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 -> /300cf3d4-e317-44c8-acd8-5f9989779c7c/4304a2bc-ba15-4549-9a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; root_uuid bd07fb41-9ea7-4d0f-b403-cbcdc979b1cd -> 300cf3d4-e317-44c8-acd8-5f9989779c7c
- C6: value 100nF -> 10nF; hierarchy_path /bd07fb41-9ea7-4d0f-b403-cbcdc979b1cd/31dca4aa-880f-4bf5-8b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 -> /300cf3d4-e317-44c8-acd8-5f9989779c7c/4304a2bc-ba15-4549-9a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; root_uuid bd07fb41-9ea7-4d0f-b403-cbcdc979b1cd -> 300cf3d4-e317-44c8-acd8-5f9989779c7c
- C7: value 1.5nF -> 100pF; hierarchy_path /bd07fb41-9ea7-4d0f-b403-cbcdc979b1cd/31dca4aa-880f-4bf5-8b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 -> /300cf3d4-e317-44c8-acd8-5f9989779c7c/4304a2bc-ba15-4549-9a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; root_uuid bd07fb41-9ea7-4d0f-b403-cbcdc979b1cd -> 300cf3d4-e317-44c8-acd8-5f9989779c7c
- C8: value 220nF -> 5.1pF; hierarchy_path /bd07fb41-9ea7-4d0f-b403-cbcdc979b1cd/31dca4aa-880f-4bf5-8b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 -> /300cf3d4-e317-44c8-acd8-5f9989779c7c/4304a2bc-ba15-4549-9a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; root_uuid bd07fb41-9ea7-4d0f-b403-cbcdc979b1cd -> 300cf3d4-e317-44c8-acd8-5f9989779c7c
- C9: value 10nF -> 5.1pF; hierarchy_path /bd07fb41-9ea7-4d0f-b403-cbcdc979b1cd/31dca4aa-880f-4bf5-8b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 -> /300cf3d4-e317-44c8-acd8-5f9989779c7c/4304a2bc-ba15-4549-9a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; root_uuid bd07fb41-9ea7-4d0f-b403-cbcdc979b1cd -> 300cf3d4-e317-44c8-acd8-5f9989779c7c
- L1: value 56nH -> 15nH; hierarchy_path /bd07fb41-9ea7-4d0f-b403-cbcdc979b1cd/31dca4aa-880f-4bf5-8b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 -> /300cf3d4-e317-44c8-acd8-5f9989779c7c/4304a2bc-ba15-4549-9a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; root_uuid bd07fb41-9ea7-4d0f-b403-cbcdc979b1cd -> 300cf3d4-e317-44c8-acd8-5f9989779c7c
- L2: value 56nH -> 43nH; hierarchy_path /bd07fb41-9ea7-4d0f-b403-cbcdc979b1cd/31dca4aa-880f-4bf5-8b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 -> /300cf3d4-e317-44c8-acd8-5f9989779c7c/4304a2bc-ba15-4549-9a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; root_uuid bd07fb41-9ea7-4d0f-b403-cbcdc979b1cd -> 300cf3d4-e317-44c8-acd8-5f9989779c7c
- L3: value 27nH -> 22nH; hierarchy_path /bd07fb41-9ea7-4d0f-b403-cbcdc979b1cd/31dca4aa-880f-4bf5-8b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 -> /300cf3d4-e317-44c8-acd8-5f9989779c7c/4304a2bc-ba15-4549-9a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; root_uuid bd07fb41-9ea7-4d0f-b403-cbcdc979b1cd -> 300cf3d4-e317-44c8-acd8-5f9989779c7c
- L4: value 27nH -> 56nH; hierarchy_path /bd07fb41-9ea7-4d0f-b403-cbcdc979b1cd/31dca4aa-880f-4bf5-8b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 -> /300cf3d4-e317-44c8-acd8-5f9989779c7c/4304a2bc-ba15-4549-9a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; root_uuid bd07fb41-9ea7-4d0f-b403-cbcdc979b1cd -> 300cf3d4-e317-44c8-acd8-5f9989779c7c
- L6: value 43nH -> 27nH; hierarchy_path /bd07fb41-9ea7-4d0f-b403-cbcdc979b1cd/31dca4aa-880f-4bf5-8b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 -> /300cf3d4-e317-44c8-acd8-5f9989779c7c/4304a2bc-ba15-4549-9a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; root_uuid bd07fb41-9ea7-4d0f-b403-cbcdc979b1cd -> 300cf3d4-e317-44c8-acd8-5f9989779c7c
- L7: value 22nH -> 56nH; hierarchy_path /bd07fb41-9ea7-4d0f-b403-cbcdc979b1cd/31dca4aa-880f-4bf5-8b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 -> /300cf3d4-e317-44c8-acd8-5f9989779c7c/4304a2bc-ba15-4549-9a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; root_uuid bd07fb41-9ea7-4d0f-b403-cbcdc979b1cd -> 300cf3d4-e317-44c8-acd8-5f9989779c7c
- L8: value 15nH -> 27nH; hierarchy_path /bd07fb41-9ea7-4d0f-b403-cbcdc979b1cd/31dca4aa-880f-4bf5-8b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 -> /300cf3d4-e317-44c8-acd8-5f9989779c7c/4304a2bc-ba15-4549-9a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; root_uuid bd07fb41-9ea7-4d0f-b403-cbcdc979b1cd -> 300cf3d4-e317-44c8-acd8-5f9989779c7c
Connections:
- net GND: now also C7.2, L6.2, C57.2, C58.2, C59.2, C60.2, C61.2, C62.2, C63.2, C64.2, R7.1; no longer C1.2, C10.2, C18.2, C2.2, C3.2, C5.2, C8.2, U1.20 (LNA_N)
- net UHF_CSN: now also R4.2
- net UHF_RESET: now also R5.2
- net UHF_AVDD_FILT renamed +3V3
- net +3V3: now also C21.1, C5.1, C6.1, C7.1, C57.1, C58.1, C59.1, C60.1, C61.1, C62.1, C63.1, C64.1, R4.1, R5.1, R6.1; no longer C10.1, C12.1, C13.1, C14.1, C15.1, C16.1, C17.1, C8.1, C9.1
- net UHF_DCPL: no longer names the net of C3.1
- net UHF_DCPL: now also C1.2, L1.2, L2.1; no longer U1.6 (DCPL)
- net UHF_DCPL_PFD: no longer names the net of U1.26 (DCPL_PFD_CHP)
- net UHF_DCPL_PFD: now also C14.1; no longer C5.1
- net UHF_DCPL_VCO: no longer names the net of U1.21 (DCPL_VCO)
- net UHF_DCPL_VCO: now also C16.1; no longer C4.1
- net UHF_DCPL_XOSC: no longer names the net of U1.29 (DCPL_XOSC)
- net UHF_DCPL_XOSC: now also C15.1; no longer C6.1
- removed net UHF_LN0: C18.1, L1.2, L2.1
- net UHF_LN1: no longer names the net of L2.2, L3.1
- net UHF_LN1: now also C4.1
- net UHF_LN2: no longer names the net of L3.2
- net UHF_LN2: now also C10.1; no longer L4.1
- removed net UHF_LN3: C21.1, L4.2, L5.1
- net UHF_LN4: no longer names the net of L5.2
- net UHF_LN4: now also C3.2, U1.18 (TRX_SW); no longer L6.1
- net UHF_LN5: no longer names the net of L7.1
- net UHF_LN5: now also C8.1, L6.1, U1.19 (LNA_P); no longer L6.2
- net UHF_LN6: no longer names the net of L7.2, L8.1
- net UHF_LN6: now also C9.1, U1.20 (LNA_N)
- removed net UHF_LN7: J1.1 (In), L8.2, U1.18 (TRX_SW), U1.19 (LNA_P)
- net UHF_LPF0: no longer names the net of U1.23 (LPF0)
- net UHF_LPF0: now also C18.2; no longer C7.1
- net UHF_LPF1: no longer names the net of U1.24 (LPF1)
- net UHF_LPF1: now also C18.1; no longer C7.2
- net UHF_MN1: no longer names the net of L1.1
- net UHF_MN1: now also C1.1, C2.2
- net UHF_PA: no longer names the net of U1.17 (PA)
- net UHF_PA: now also C2.1, L4.2
- net UHF_RBIAS: no longer names the net of U1.14 (RBIAS)
- net UHF_RBIAS: now also R7.2
- net UHF_XOSC_Q1: no longer names the net of U1.30 (XOSC_Q1), Y1.1
- net UHF_XOSC_Q1: now also C12.1; no longer C1.1
- net UHF_XOSC_Q2: no longer names the net of U1.31 (XOSC_Q2), Y1.3
- net UHF_XOSC_Q2: now also C13.1; no longer C2.1
- new net: C17.1, U1.6 (DCPL)
- new net: C10.2, J1.1 (In)
- new net: C8.2, L5.1, L8.2
- new net: C5.2, L4.1, R6.2
Other:
- note added: "CC1200 UHF 432 MHz Matching Network Source: M17 CC1200_HAT Rev B (SP5WWP/DB9MAT) Cross-ref: TI SWRR122 (CC1200EM 420-470 MHz) All RF matching values are exact copies from the M17 verified design (+14 dBm at 433.475 MHz). 3-path topology sharing single SMA antenna: TX: PA → C2-L1-C1-L2-C3-L3-C4 → C10(DC block) → SMA TRX: TRX_SW → C3 to TX path, L5 to balun center RX: LNA_P/N differential balun (L6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"

Commit message: did final routing and added Farnell and LCSC numbers to all components
Parts:
- C1: Farnell (none) -> 1813415; LCSC (none) -> C1651
- C10: Farnell (none) -> 2496882; LCSC (none) -> C342910
- C12, C13: Farnell (none) -> 721980; LCSC (none) -> C1644
- C14, C15, C21, C57, C58, C59, C60, C61, C62, C63, C64: Farnell (none) -> 2495363; LCSC (none) -> C1622
- C16, C6: Farnell (none) -> 1759022; LCSC (none) -> C57112
- C17: Farnell (none) -> 1828900; LCSC (none) -> C21120
- C18: Farnell (none) -> 2672137; LCSC (none) -> C76600
- C2: Farnell (none) -> 2280868; LCSC (none) -> C445758
- C3, C8, C9: Farnell (none) -> 2904766; LCSC (none) -> C61816
- C4: Farnell (none) -> 3759543; LCSC (none) -> C48579262
- C5: Farnell (none) -> 1572627; LCSC (none) -> C338104
- C7: Farnell (none) -> 722080; LCSC (none) -> C14858
- J1: Farnell (none) -> 2112467
- L1, L5: Farnell (none) -> 1515375; LCSC (none) -> C23651
- L2: Farnell (none) -> 2470386; LCSC (none) -> C29683
- L3: Farnell (none) -> 1515382; LCSC (none) -> C98071
- L4, L7: Farnell (none) -> 3354667; LCSC (none) -> C12831
- L6, L8: Farnell (none) -> 1515383; LCSC (none) -> C162550
- R4, R5: Farnell (none) -> 9238603; LCSC (none) -> C25804
- R6: Farnell (none) -> 9238271; LCSC (none) -> C245924
- R7: Farnell (none) -> 9238697; LCSC (none) -> C23206
- U1: Farnell (none) -> 2345430; LCSC (none) -> C122881
- Y1: Farnell (none) -> 1712847; LCSC (none) -> C5380316
