File: MOTOR_RF_HAT/gyro.kicad_sch (KiCad schematic)
At the start: 0 parts

Commit message: MOTOR_RF_HAT: fix TestPoint:smallpad → components:smallpad in solder_pads
All 18 test point footprint references in solder_pads.kicad_sch now
point to the local components:smallpad instead of TestPoint:smallpad
(which doesn't exist in KiCad's global TestPoint library).

Co-Authored-By: Claude Opus 4.6 (1M context) <noreply@anthropic.com>
Other:
- note removed: "add breakout pads"
