File: MOTOR_RF_HAT/Pi_Header.kicad_sch (KiCad schematic)
At the start: 1 part, among them J3 Raspberry_Pi_2_3

Commit message: MOTOR_RF_HAT: port full RF_HAT project with all libs localized
Copied complete RF_HAT_out KiCad project (schematic + PCB layout +
4 hierarchical sub-sheets) as the base for the combined board.

Changes from original RF_HAT:
- Renamed RF_HAT → MOTOR_RF_HAT in all project/schematic references
- Imported LMR51420YDDCR + XRTC303020D4R7MBCA symbols from personal
  lib into project-local components.kicad_sym
- Copied corresponding footprints + 3D models (SOT-23-6, inductor)
  into components.pretty/ and components.3dshapes/
- Fixed all lib: → components: references in schematics and PCB
- Removed reference/ directory (schematics are now live sub-sheets)
- ERC: 20 violations (19 pre-existing from RF_HAT + 1 from rename)
- Zero external library dependencies — fully self-contained

Ready to add motor driver (A4950E), encoder, and IMU (ADXL345)
sub-sheets. Existing CC1200 UHF/VHF, Pi header, Pico, power,
NeoPixel, and buzzer circuits carry over unchanged.

Co-Authored-By: Claude Opus 4.6 (1M context) <noreply@anthropic.com>
Parts:
- J3: project_name RF_HAT -> MOTOR_RF_HAT
Other:
- title: RF_HAT -> MOTOR_RF_HAT
Changed lines of the file:
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@@
 	(paper "A3")
 	(title_block
-		(title "RF_HAT")
+		(title "MOTOR_RF_HAT")
 	)
 	(text_box "Raspberry Pi 40-pin GPIO header - UART passthrough"
@@
 		)
 		(instances
-			(project "RF_HAT"
+			(project "MOTOR_RF_HAT"
 				(path "/300cf3d4-e317-44c8-acd8-5f9989779c7c/df2c4ae5-dfcc-4b06-a511-feaff2e2867e"
 					(reference "#PWR041")
@@
 			)
 		)
-		(property "project_name" "RF_HAT"
+		(property "project_name" "MOTOR_RF_HAT"
 			(at 53.34 71.1199 0)
 			(effects
