File: MOTOR_RF_HAT/solder_pads.kicad_sch (KiCad schematic)
At the start: 18 parts

Commit message: MOTOR_RF_HAT: localize all libraries — zero external dependencies
- Extracted smallpad footprint from MotorPCB PCB into local lib
- Extracted TB6642FG (HSOP-16) footprint from MotorPCB PCB into local lib
- Extracted TB6642FG_8_EL symbol from MotorPCB schematic into local lib
- Fixed all references: TestPoint:smallpad → components:smallpad,
  easyeda2kicad:TB6642FG → components:TB6642FG_8_EL,
  easyeda2kicad:HSOP-16 → components:HSOP-16

All schematic lib_id references now resolve to either:
  - components: (project-local)
  - KiCad globals (Device, Connector, RF, power, etc.)

Local lib now contains 7 symbols:
  S2B-XH-A-(LF)(SN), S6B-XH-A_(LF)(SN), XT30PW-M, A4950E,
  LMR51420YDDCR, XRTC303020D4R7MBCA, TB6642FG_8_EL

Co-Authored-By: Claude Opus 4.6 (1M context) <noreply@anthropic.com>
Parts:
- TP1, TP10, TP11, TP12, TP13, TP14, TP15, TP16, TP17, TP18, TP2, TP3, TP4, TP5, TP6, TP7, TP8, TP9: footprint TestPoint:smallpad -> components:smallpad
Changed lines of the file:
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@@
 			)
 		)
-		(property "Footprint" "TestPoint:smallpad"
+		(property "Footprint" "components:smallpad"
 			(at 87.63 48.26 0)
 			(effects
@@
 			)
 		)
-		(property "Footprint" "TestPoint:smallpad"
+		(property "Footprint" "components:smallpad"
 			(at 87.63 92.71 0)
 			(effects
@@
 			)
 		)
-		(property "Footprint" "TestPoint:smallpad"
+		(property "Footprint" "components:smallpad"
 			(at 87.63 58.42 0)
 			(effects
@@
 			)
 		)
-		(property "Footprint" "TestPoint:smallpad"
+		(property "Footprint" "components:smallpad"
 			(at 87.63 50.8 0)
 			(effects
@@
 			)
 		)
-		(property "Footprint" "TestPoint:smallpad"
+		(property "Footprint" "components:smallpad"
 			(at 87.63 25.4 0)
 			(effects
@@
 			)
 		)
-		(property "Footprint" "TestPoint:smallpad"
+		(property "Footprint" "components:smallpad"
 			(at 87.63 85.09 0)
 			(effects
@@
 			)
 		)
-		(property "Footprint" "TestPoint:smallpad"
+		(property "Footprint" "components:smallpad"
 			(at 87.63 82.55 0)
 			(effects
@@
 			)
 		)
-		(property "Footprint" "TestPoint:smallpad"
+		(property "Footprint" "components:smallpad"
 			(at 87.63 27.94 0)
 			(effects
@@
 			)
 		)
-		(property "Footprint" "TestPoint:smallpad"
+		(property "Footprint" "components:smallpad"
 			(at 87.63 30.48 0)
 			(effects
@@
 			)
 		)
-		(property "Footprint" "TestPoint:smallpad"
+		(property "Footprint" "components:smallpad"
 			(at 87.63 87.63 0)
 			(effects
@@
 			)
 		)
-		(property "Footprint" "TestPoint:smallpad"
+		(property "Footprint" "components:smallpad"
 			(at 87.63 95.25 0)
 			(effects
@@
 			)
 		)
-		(property "Footprint" "TestPoint:smallpad"
+		(property "Footprint" "components:smallpad"
 			(at 87.63 77.47 0)
 			(effects
@@
 			)
 		)
-		(property "Footprint" "TestPoint:smallpad"
+		(property "Footprint" "components:smallpad"
 			(at 87.63 55.88 0)
 			(effects
@@
 			)
 		)
-		(property "Footprint" "TestPoint:smallpad"
+		(property "Footprint" "components:smallpad"
 			(at 87.63 90.17 0)
 			(effects
@@
 			)
 		)
-		(property "Footprint" "TestPoint:smallpad"
+		(property "Footprint" "components:smallpad"
 			(at 87.63 53.34 0)
 			(effects
@@
 			)
 		)
-		(property "Footprint" "TestPoint:smallpad"
+		(property "Footprint" "components:smallpad"
 			(at 87.63 33.02 0)
 			(effects
@@
 			)
 		)
-		(property "Footprint" "TestPoint:smallpad"
+		(property "Footprint" "components:smallpad"
 			(at 87.63 35.56 0)
 			(effects
@@
 			)
 		)
-		(property "Footprint" "TestPoint:smallpad"
+		(property "Footprint" "components:smallpad"
 			(at 87.63 80.01 0)
 			(effects

Commit message: MOTOR_RF_HAT: assign components:smallpad to all TestPoint_Small
Assigned local smallpad footprint to 8 TestPoint_Small instances:
- 7 in solder_pads.kicad_sch
- 1 in root schematic (TP19)

Co-Authored-By: Claude Opus 4.6 (1M context) <noreply@anthropic.com>
Parts:
- TP1, TP10, TP11, TP12, TP13, TP14, TP15, TP16, TP17, TP18, TP2, TP3, TP4, TP5, TP6, TP7, TP8, TP9: value ~ -> (none)

Commit message: MOTOR_RF_HAT: add TestPoint lib alias to fix persistent smallpad errors
KiCad's lib_symbols cache keeps reverting footprint refs to
TestPoint:smallpad on save. Added TestPoint as a footprint library
alias pointing to components.pretty so both TestPoint:smallpad and
components:smallpad resolve to the same local footprint.

Co-Authored-By: Claude Opus 4.6 (1M context) <noreply@anthropic.com>
Parts:
- renumbered TP9 to TP11, TP8 to TP12, TP7 to TP13, TP5 to TP14, TP4 to TP15, TP3 to TP16, TP2 to TP17, TP1 to TP18, TP6 to TP19, TP18 to TP2, TP17 to TP3, TP16 to TP4, TP15 to TP5, TP14 to TP6, TP13 to TP7, TP12 to TP8, TP11 to TP9
Changed lines of the file:
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@@
 		(dnp no)
 		(fields_autoplaced yes)
-		(property "Reference" "#PWR011"
+		(property "Reference" "#PWR075"
 			(at 54.61 93.98 0)
 			(hide yes)
@@
 			(project "MOTOR_RF_HAT"
 				(path "/300cf3d4-e317-44c8-acd8-5f9989779c7c/897cf420-fdd5-435e-b081-e1fa633c20b5"
-					(reference "#PWR011")
+					(reference "#PWR075")
 					(unit 1)
 				)
@@
 		(in_pos_files yes)
 		(dnp no)
-		(property "Reference" "TP13"
+		(property "Reference" "TP7"
 			(at 83.566 48.26 0)
 			(show_name no)
@@
 			(project "MOTOR_RF_HAT"
 				(path "/300cf3d4-e317-44c8-acd8-5f9989779c7c/897cf420-fdd5-435e-b081-e1fa633c20b5"
-					(reference "TP13")
+					(reference "TP7")
 					(unit 1)
 				)
@@
 		(dnp no)
 		(fields_autoplaced yes)
-		(property "Reference" "#PWR09"
+		(property "Reference" "#PWR081"
 			(at 80.01 67.31 0)
 			(hide yes)
@@
 			(project "MOTOR_RF_HAT"
 				(path "/300cf3d4-e317-44c8-acd8-5f9989779c7c/897cf420-fdd5-435e-b081-e1fa633c20b5"
-					(reference "#PWR09")
+					(reference "#PWR081")
 					(unit 1)
 				)
@@
 		(in_pos_files yes)
 		(dnp no)
-		(property "Reference" "TP1"
+		(property "Reference" "TP18"
 			(at 83.566 92.71 0)
 			(show_name no)
@@
 			(project "MOTOR_RF_HAT"
 				(path "/300cf3d4-e317-44c8-acd8-5f9989779c7c/897cf420-fdd5-435e-b081-e1fa633c20b5"
-					(reference "TP1")
+					(reference "TP18")
 					(unit 1)
 				)
@@
 		(in_pos_files yes)
 		(dnp no)
-		(property "Reference" "TP9"
+		(property "Reference" "TP11"
 			(at 83.566 58.42 0)
 			(show_name no)
@@
 			(project "MOTOR_RF_HAT"
 				(path "/300cf3d4-e317-44c8-acd8-5f9989779c7c/897cf420-fdd5-435e-b081-e1fa633c20b5"
-					(reference "TP9")
+					(reference "TP11")
 					(unit 1)
 				)
@@
 		(in_pos_files yes)
 		(dnp no)
-		(property "Reference" "TP12"
+		(property "Reference" "TP8"
 			(at 83.566 50.8 0)
 			(show_name no)
@@
 			(project "MOTOR_RF_HAT"
 				(path "/300cf3d4-e317-44c8-acd8-5f9989779c7c/897cf420-fdd5-435e-b081-e1fa633c20b5"
-					(reference "TP12")
+					(reference "TP8")
 					(unit 1)
 				)
@@
 		(in_pos_files yes)
 		(dnp no)
-		(property "Reference" "TP18"
+		(property "Reference" "TP2"
 			(at 83.566 25.4 0)
 			(show_name no)
@@
 			(project "MOTOR_RF_HAT"
 				(path "/300cf3d4-e317-44c8-acd8-5f9989779c7c/897cf420-fdd5-435e-b081-e1fa633c20b5"
-					(reference "TP18")
+					(reference "TP2")
 					(unit 1)
 				)
@@
 		(in_pos_files yes)
 		(dnp no)
-		(property "Reference" "TP4"
+		(property "Reference" "TP15"
 			(at 83.566 85.09 0)
 			(show_name no)
@@
 			(project "MOTOR_RF_HAT"
 				(path "/300cf3d4-e317-44c8-acd8-5f9989779c7c/897cf420-fdd5-435e-b081-e1fa633c20b5"
-					(reference "TP4")
+					(reference "TP15")
 					(unit 1)
 				)
@@
 		(dnp no)
 		(fields_autoplaced yes)
-		(property "Reference" "#PWR065"
+		(property "Reference" "#PWR080"
 			(at 80.01 44.45 0)
 			(hide yes)
@@
 			(project "MOTOR_RF_HAT"
 				(path "/300cf3d4-e317-44c8-acd8-5f9989779c7c/897cf420-fdd5-435e-b081-e1fa633c20b5"
-					(reference "#PWR065")
+					(reference "#PWR080")
 					(unit 1)
 				)
@@
 		(dnp no)
 		(fields_autoplaced yes)
-		(property "Reference" "#PWR012"
+		(property "Reference" "#PWR082"
 			(at 80.01 104.14 0)
 			(hide yes)
@@
 			(project "MOTOR_RF_HAT"
 				(path "/300cf3d4-e317-44c8-acd8-5f9989779c7c/897cf420-fdd5-435e-b081-e1fa633c20b5"
-					(reference "#PWR012")
+					(reference "#PWR082")
 					(unit 1)
 				)
@@
 		(in_pos_files yes)
 		(dnp no)
-		(property "Reference" "TP5"
+		(property "Reference" "TP14"
 			(at 83.566 82.55 0)
 			(show_name no)
@@
 			(project "MOTOR_RF_HAT"
 				(path "/300cf3d4-e317-44c8-acd8-5f9989779c7c/897cf420-fdd5-435e-b081-e1fa633c20b5"
-					(reference "TP5")
+					(reference "TP14")
 					(unit 1)
 				)
@@
 		(in_pos_files yes)
 		(dnp no)
-		(property "Reference" "TP17"
+		(property "Reference" "TP3"
 			(at 83.566 27.94 0)
 			(show_name no)
@@
 			(project "MOTOR_RF_HAT"
 				(path "/300cf3d4-e317-44c8-acd8-5f9989779c7c/897cf420-fdd5-435e-b081-e1fa633c20b5"
-					(reference "TP17")
+					(reference "TP3")
 					(unit 1)
 				)
@@
 		(in_pos_files yes)
 		(dnp no)
-		(property "Reference" "TP16"
+		(property "Reference" "TP4"
 			(at 83.566 30.48 0)
 			(show_name no)
@@
 			(project "MOTOR_RF_HAT"
 				(path "/300cf3d4-e317-44c8-acd8-5f9989779c7c/897cf420-fdd5-435e-b081-e1fa633c20b5"
-					(reference "TP16")
+					(reference "TP4")
 					(unit 1)
 				)
@@
 		(dnp no)
 		(fields_autoplaced yes)
-		(property "Reference" "#PWR068"
+		(property "Reference" "#PWR076"
 			(at 59.69 34.29 0)
 			(hide yes)
@@
 			(project "MOTOR_RF_HAT"
 				(path "/300cf3d4-e317-44c8-acd8-5f9989779c7c/897cf420-fdd5-435e-b081-e1fa633c20b5"
-					(reference "#PWR068")
+					(reference "#PWR076")
 					(unit 1)
 				)
@@
 		(in_pos_files yes)
 		(dnp no)
-		(property "Reference" "TP3"
+		(property "Reference" "TP16"
 			(at 83.566 87.63 0)
 			(show_name no)
@@
 			(project "MOTOR_RF_HAT"
 				(path "/300cf3d4-e317-44c8-acd8-5f9989779c7c/897cf420-fdd5-435e-b081-e1fa633c20b5"
-					(reference "TP3")
+					(reference "TP16")
 					(unit 1)
 				)
@@
 		(dnp no)
 		(fields_autoplaced yes)
-		(property "Reference" "#PWR066"
+		(property "Reference" "#PWR078"
 			(at 67.31 34.29 0)
 			(hide yes)
@@
 			(project "MOTOR_RF_HAT"
 				(path "/300cf3d4-e317-44c8-acd8-5f9989779c7c/897cf420-fdd5-435e-b081-e1fa633c20b5"
-					(reference "#PWR066")
+					(reference "#PWR078")
 					(unit 1)
 				)
@@
 		(in_pos_files yes)
 		(dnp no)
-		(property "Reference" "TP6"
+		(property "Reference" "TP19"
 			(at 83.566 95.25 0)
 			(show_name no)
@@
 			(project "MOTOR_RF_HAT"
 				(path "/300cf3d4-e317-44c8-acd8-5f9989779c7c/897cf420-fdd5-435e-b081-e1fa633c20b5"
-					(reference "TP6")
+					(reference "TP19")
 					(unit 1)
 				)
@@
 		(in_pos_files yes)
 		(dnp no)
-		(property "Reference" "TP8"
+		(property "Reference" "TP12"
 			(at 83.566 77.47 0)
 			(show_name no)
@@
 			(project "MOTOR_RF_HAT"
 				(path "/300cf3d4-e317-44c8-acd8-5f9989779c7c/897cf420-fdd5-435e-b081-e1fa633c20b5"
-					(reference "TP8")
+					(reference "TP12")
 					(unit 1)
 				)
@@
 		(dnp no)
 		(fields_autoplaced yes)
-		(property "Reference" "#PWR07"
+		(property "Reference" "#PWR077"
 			(at 59.69 57.15 0)
 			(hide yes)
@@
 			(project "MOTOR_RF_HAT"
 				(path "/300cf3d4-e317-44c8-acd8-5f9989779c7c/897cf420-fdd5-435e-b081-e1fa633c20b5"
-					(reference "#PWR07")
+					(reference "#PWR077")
 					(unit 1)
 				)
@@
 		(in_pos_files yes)
 		(dnp no)
-		(property "Reference" "TP2"
+		(property "Reference" "TP17"
 			(at 83.566 90.17 0)
 			(show_name no)
@@
 			(project "MOTOR_RF_HAT"
 				(path "/300cf3d4-e317-44c8-acd8-5f9989779c7c/897cf420-fdd5-435e-b081-e1fa633c20b5"
-					(reference "TP2")
+					(reference "TP17")
 					(unit 1)
 				)
@@
 		(in_pos_files yes)
 		(dnp no)
-		(property "Reference" "TP11"
+		(property "Reference" "TP9"
 			(at 83.566 53.34 0)
 			(show_name no)
@@
 			(project "MOTOR_RF_HAT"
 				(path "/300cf3d4-e317-44c8-acd8-5f9989779c7c/897cf420-fdd5-435e-b081-e1fa633c20b5"
-					(reference "TP11")
+					(reference "TP9")
 					(unit 1)
 				)
@@
 		(in_pos_files yes)
 		(dnp no)
-		(property "Reference" "TP15"
+		(property "Reference" "TP5"
 			(at 83.566 33.02 0)
 			(show_name no)
@@
 			(project "MOTOR_RF_HAT"
 				(path "/300cf3d4-e317-44c8-acd8-5f9989779c7c/897cf420-fdd5-435e-b081-e1fa633c20b5"
-					(reference "TP15")
+					(reference "TP5")
 					(unit 1)
 				)
@@
 		(dnp no)
 		(fields_autoplaced yes)
-		(property "Reference" "#PWR08"
+		(property "Reference" "#PWR079"
 			(at 67.31 57.15 0)
 			(hide yes)
@@
 			(project "MOTOR_RF_HAT"
 				(path "/300cf3d4-e317-44c8-acd8-5f9989779c7c/897cf420-fdd5-435e-b081-e1fa633c20b5"
-					(reference "#PWR08")
+					(reference "#PWR079")
 					(unit 1)
 				)
@@
 		(in_pos_files yes)
 		(dnp no)
-		(property "Reference" "TP14"
+		(property "Reference" "TP6"
 			(at 83.566 35.56 0)
 			(show_name no)
@@
 			(project "MOTOR_RF_HAT"
 				(path "/300cf3d4-e317-44c8-acd8-5f9989779c7c/897cf420-fdd5-435e-b081-e1fa633c20b5"
-					(reference "TP14")
+					(reference "TP6")
 					(unit 1)
 				)
@@
 		(dnp no)
 		(fields_autoplaced yes)
-		(property "Reference" "#PWR010"
+		(property "Reference" "#PWR074"
 			(at 46.99 93.98 0)
 			(hide yes)
@@
 			(project "MOTOR_RF_HAT"
 				(path "/300cf3d4-e317-44c8-acd8-5f9989779c7c/897cf420-fdd5-435e-b081-e1fa633c20b5"
-					(reference "#PWR010")
+					(reference "#PWR074")
 					(unit 1)
 				)
@@
 		(in_pos_files yes)
 		(dnp no)
-		(property "Reference" "TP7"
+		(property "Reference" "TP13"
 			(at 83.566 80.01 0)
 			(show_name no)
@@
 			(project "MOTOR_RF_HAT"
 				(path "/300cf3d4-e317-44c8-acd8-5f9989779c7c/897cf420-fdd5-435e-b081-e1fa633c20b5"
-					(reference "TP7")
-					(unit 1)
-				)
+					(reference "TP13")
+					(unit 1)
+				)

Commit message: MOTOR_RF_HAT: 0805→0603 passives, encoder caps 100nF→100pF
- Changed all capacitor and resistor footprints from 0805 to 0603
  across all schematic sheets (CC1200 UHF/VHF, root, azimuth,
  elevation, encoders)
- Fixed encoder RC filter caps C68-C71 from 100nF to 100pF
  (fc = 15.9 MHz, transparent to 35 kHz encoder signal)

Co-Authored-By: Claude Opus 4.6 (1M context) <noreply@anthropic.com>
Parts:
- removed TP10, TP11, TP12, TP13, TP14, TP15, TP16, TP17, TP18, TP19, TP2, TP3, TP4, TP5, TP6, TP7, TP8, TP9: (no value), components:smallpad, symbol Connector:TestPoint_Small
