File: MOTOR_RF_HAT/MOTOR_RF_HAT.kicad_pcb (KiCad board)
At the start: 6 copper layers, 56 x 65 mm, 135 parts, among them J1 Conn_01x01, J2 Conn_01x01, J3 Raspberry_Pi_2_3, J4 SMA, J5 SMA, J6 JST_AZ, J7 JST_EL, Q1 BSS138, U1 XT30PW-M, U2 LMR51420YFDDCR, U3 CC1200RHBR, U4 RaspberryPi_Pico, U5 CC1200RHBR, U6 A4950E, U7 A4950E, Y1 40MHz, Y2 40MHz

Commit message: MOTOR_RF_HAT: final production check — BOM fix + routed PCB
BOM fix:
- A4950 VBB bypass caps (C60-C62, C64-C66): changed MPN from
  CL10A106KP8NNNC (10uF/10V 0603, WRONG) to CL21A106KPFNNNE
  (10uF/10V 0805). Note: for 24V bus these should ideally be
  50V-rated — verify before ordering.

ERC: 47 violations (4 errors, 43 warnings)
- All 4 errors are false positives (power pin connectivity
  through Schottky diode, Pico dual-ground, cross-sheet power)
- 43 warnings are pre-existing from RF_HAT base design

Production readiness:
- All symbols resolve (5 local + 15 KiCad global)
- All footprints resolve (5 local + 19 KiCad global)
- All 3D models resolve (20 in PCB, 9 in footprints)
- BOM enriched: 122/131 components have LCSC + MPN + Farnell
- Firmware builds clean: 5.7% RAM, 4.2% flash

Before ordering:
- [ ] Run Update PCB from Schematic (new motor/encoder nets)
- [ ] Verify A4950 VBB cap voltage rating (need 50V for 24V bus)
- [ ] Add bulk 470µF electrolytic externally
- [ ] VNA tune VHF matching network post-assembly

Co-Authored-By: Claude Opus 4.6 (1M context) <noreply@anthropic.com>
Parts:
- C68, C69, C70, C71, R11, R12, R13, R14: moved to B.Cu
- moved TP1 52.5 mm to (166.0, 118.6)
- moved D1 52.3 mm to (188.4, 76.4), turned to 90 degrees
- moved C68 48.9 mm to (165.2, 98.8), turned to 180 degrees
- moved C70 47.1 mm to (165.2, 101.3), turned to 180 degrees
- moved R11 46.6 mm to (168.2, 98.8), turned to 180 degrees
- moved R13 45.7 mm to (168.2, 101.3), turned to 180 degrees
- moved R14 44.9 mm to (167.9, 85.8), turned to 180 degrees
- moved R12 44.4 mm to (167.9, 83.9), turned to 180 degrees
- moved C69 42.0 mm to (164.9, 83.9), turned to 180 degrees
- moved C71 41.4 mm to (164.9, 85.7), turned to 180 degrees
- moved R2 0.73 mm to (205.5, 80.5), turned to 180 degrees
- moved R1 0.54 mm to (205.1, 73.4), turned to 0 degrees
Connections:
- C4 pad 1: +3V3 -> /4.5V
- C5 pad 1: +3V3 -> /4.5V
- C6 pad 1: +3V3 -> /4.5V
- C7 pad 1: +3V3 -> /4.5V
- U4 pad 6: /Pico_SPI_Host/WS2812 -> /WS2812B
Routing:
- net /Encoders/AZ_ENC_A: track 0.00 -> 73.7 mm
- net /Encoders/EL_ENC_A: track 0.00 -> 69.7 mm
- net (no net): track 38.4 -> 0.00 mm, vias 3 -> 0
- net /Azimuth/AZ_EN/IN1: track 0.00 -> 36.3 mm, vias 0 -> 1
- net /Encoders/EL_ENC_B: track 9.16 -> 41.1 mm, vias 1 -> 0
- net /Azimuth/AZ_PH/IN2: track 0.00 -> 31.9 mm, vias 0 -> 1
- net /Pico_SPI_Host/IMU_CS: track 0.00 -> 31.4 mm, vias 0 -> 1
- net /Pico_SPI_Host/BUZZER: track 36.7 -> 64.4 mm, vias 1 -> 3
- net /4.5V: track 0.00 -> 27.1 mm
- net GND: track 48.8 -> 75.6 mm, vias 62 -> 137
- net /CC1200_VHF_144MHz/VHF_MOSI: track 6.12 -> 29.5 mm, vias 2 -> 3
- net /CC1200_VHF_144MHz/VHF_SCLK: track 8.31 -> 31.6 mm, vias 2 -> 3
- net /CC1200_VHF_144MHz/VHF_MISO: track 15.6 -> 38.4 mm
- net /Elevation/EL_EN/IN1: track 0.00 -> 20.9 mm, vias 0 -> 1
- net /Encoders/AZ_ENC_B: track 7.66 -> 22.9 mm, vias 2 -> 1
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- added copper zone on B.Cu, net +24V
- added copper zone on F.Cu, net +24V
- added copper zone on B.Cu, net GND
- added copper zone on In2.Cu, net GND
- added copper zone on In3.Cu, net GND
