File: MOTOR_RF_HAT/Pico_SPI_Host.kicad_sch (KiCad schematic)
At the start: 1 part, among them U3 RaspberryPi_Pico

Commit message: MOTOR_RF_HAT: port full RF_HAT project with all libs localized
Copied complete RF_HAT_out KiCad project (schematic + PCB layout +
4 hierarchical sub-sheets) as the base for the combined board.

Changes from original RF_HAT:
- Renamed RF_HAT → MOTOR_RF_HAT in all project/schematic references
- Imported LMR51420YDDCR + XRTC303020D4R7MBCA symbols from personal
  lib into project-local components.kicad_sym
- Copied corresponding footprints + 3D models (SOT-23-6, inductor)
  into components.pretty/ and components.3dshapes/
- Fixed all lib: → components: references in schematics and PCB
- Removed reference/ directory (schematics are now live sub-sheets)
- ERC: 20 violations (19 pre-existing from RF_HAT + 1 from rename)
- Zero external library dependencies — fully self-contained

Ready to add motor driver (A4950E), encoder, and IMU (ADXL345)
sub-sheets. Existing CC1200 UHF/VHF, Pi header, Pico, power,
NeoPixel, and buzzer circuits carry over unchanged.

Co-Authored-By: Claude Opus 4.6 (1M context) <noreply@anthropic.com>
Parts:
- U3: project_name RF_HAT -> MOTOR_RF_HAT
Other:
- title: RF_HAT -> MOTOR_RF_HAT
Changed lines of the file:
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@@
 	(paper "A3")
 	(title_block
-		(title "RF_HAT")
+		(title "MOTOR_RF_HAT")
 	)
 	(no_connect
@@
 			)
 		)
-		(property "project_name" "RF_HAT"
+		(property "project_name" "MOTOR_RF_HAT"
 			(at 109.22 92.7099 0)
 			(effects
@@
 		)
 		(instances
-			(project "RF_HAT"
+			(project "MOTOR_RF_HAT"
 				(path "/300cf3d4-e317-44c8-acd8-5f9989779c7c/3e644d4e-3c70-4dba-b47a-c0e6db07080d"
 					(reference "#PWR040")
@@
 		)
 		(instances
-			(project "RF_HAT"
+			(project "MOTOR_RF_HAT"
 				(path "/300cf3d4-e317-44c8-acd8-5f9989779c7c/3e644d4e-3c70-4dba-b47a-c0e6db07080d"
 					(reference "#PWR019")

Commit message: MOTOR_RF_HAT: add TestPoint lib alias to fix persistent smallpad errors
KiCad's lib_symbols cache keeps reverting footprint refs to
TestPoint:smallpad on save. Added TestPoint as a footprint library
alias pointing to components.pretty so both TestPoint:smallpad and
components:smallpad resolve to the same local footprint.

Co-Authored-By: Claude Opus 4.6 (1M context) <noreply@anthropic.com>
Parts:
- renumbered U3 to U4
Connections:
- net AZ_ENC_A: now reaches U4.19 (GPIO14)
- net AZ_ENC_B: now reaches U4.20 (GPIO15)
- net AZ_IN1: now reaches U4.4 (GPIO2)
- net AZ_IN2: now reaches U4.5 (GPIO3)
- no-connect marks 9 -> 5
Changed lines of the file:
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@@
-	)
-	(no_connect
-		(at 83.82 77.47)
-	)
-	(no_connect
-		(at 83.82 110.49)
 	)
 	(no_connect
@@
 	)
 	(no_connect
-		(at 83.82 107.95)
-	)
-	(no_connect
 		(at 83.82 67.31)
-	)
-	(no_connect
-		(at 83.82 80.01)
 	)
 	(wire
@@
 		)
 	)
+	(hierarchical_label "AZ_ENC_A"
+		(shape input)
+		(at 83.82 107.95 180)
+		(effects
+			(font
+				(size 1.27 1.27)
+			)
+			(justify right)
+		)
+	)
 	(hierarchical_label "VHF_GPIO0"
 		(shape input)
@@
 		)
 	)
+	(hierarchical_label "AZ_ENC_B"
+		(shape input)
+		(at 83.82 110.49 180)
+		(effects
+			(font
+				(size 1.27 1.27)
+			)
+			(justify right)
+		)
+	)
 	(hierarchical_label "VHF_GPIO2"
 		(shape input)
@@
 		)
 	)
+	(hierarchical_label "AZ_IN1"
+		(shape input)
+		(at 83.82 77.47 180)
+		(effects
+			(font
+				(size 1.27 1.27)
+			)
+			(justify right)
+		)
+	)
 	(hierarchical_label "UART_RX"
 		(shape input)
@@
 			)
 			(justify left)
+		)
+	)
+	(hierarchical_label "AZ_IN2"
+		(shape input)
+		(at 83.82 80.01 180)
+		(effects
+			(font
+				(size 1.27 1.27)
+			)
+			(justify right)
 		)
 	)
@@
 		(in_pos_files yes)
 		(dnp no)
-		(property "Reference" "U3"
+		(property "Reference" "U4"
 			(at 87.63 123.19 0)
 			(show_name no)
@@
 			(project "MOTOR_RF_HAT"
 				(path "/300cf3d4-e317-44c8-acd8-5f9989779c7c/3e644d4e-3c70-4dba-b47a-c0e6db07080d"
-					(reference "U3")
+					(reference "U4")
 					(unit 1)
 				)
@@
 		(dnp no)
 		(fields_autoplaced yes)
-		(property "Reference" "#PWR020"
+		(property "Reference" "#PWR040"
 			(at 111.76 53.34 0)
 			(hide yes)
@@
 			(project "MOTOR_RF_HAT"
 				(path "/300cf3d4-e317-44c8-acd8-5f9989779c7c/3e644d4e-3c70-4dba-b47a-c0e6db07080d"
-					(reference "#PWR020")
+					(reference "#PWR040")
 					(unit 1)
 				)
@@
 		(dnp no)
 		(fields_autoplaced yes)
-		(property "Reference" "#PWR040"
+		(property "Reference" "#PWR042"
 			(at 135.89 110.49 0)
 			(hide yes)
@@
 			(project "MOTOR_RF_HAT"
 				(path "/300cf3d4-e317-44c8-acd8-5f9989779c7c/3e644d4e-3c70-4dba-b47a-c0e6db07080d"
-					(reference "#PWR040")
+					(reference "#PWR042")
 					(unit 1)
 				)
@@
 		(dnp no)
 		(fields_autoplaced yes)
-		(property "Reference" "#PWR019"
+		(property "Reference" "#PWR038"
 			(at 106.68 49.53 0)
 			(hide yes)
@@
 			(project "MOTOR_RF_HAT"
 				(path "/300cf3d4-e317-44c8-acd8-5f9989779c7c/3e644d4e-3c70-4dba-b47a-c0e6db07080d"
-					(reference "#PWR019")
+					(reference "#PWR038")
 					(unit 1)
 				)
@@
 		(dnp no)
 		(fields_autoplaced yes)
-		(property "Reference" "#PWR018"
+		(property "Reference" "#PWR037"
 			(at 101.6 53.34 0)
 			(hide yes)
@@
 			(project "MOTOR_RF_HAT"
 				(path "/300cf3d4-e317-44c8-acd8-5f9989779c7c/3e644d4e-3c70-4dba-b47a-c0e6db07080d"
-					(reference "#PWR018")
+					(reference "#PWR037")
 					(unit 1)
 				)

Commit message: MOTOR_RF_HAT: 0805→0603 passives, encoder caps 100nF→100pF
- Changed all capacitor and resistor footprints from 0805 to 0603
  across all schematic sheets (CC1200 UHF/VHF, root, azimuth,
  elevation, encoders)
- Fixed encoder RC filter caps C68-C71 from 100nF to 100pF
  (fc = 15.9 MHz, transparent to 35 kHz encoder signal)

Co-Authored-By: Claude Opus 4.6 (1M context) <noreply@anthropic.com>
Connections:
- net EL_IN1: now reaches U4.32 (GPIO27_ADC1)
- net EL_IN2: now reaches U4.34 (GPIO28_ADC2)
- net +5V: no longer names the net of U4.39 (VSYS)
- net UHF_GPIO2: no longer names the net of U4.12 (GPIO9)
- net UHF_GPIO3: no longer names the net of U4.9 (GPIO6)
- net VHF_GPIO0 renamed EL_ENC_B
- net VHF_GPIO2 renamed EL_ENC_A
- net VHF_GPIO3 renamed IMU_CS
- no-connect marks 5 -> 6
Changed lines of the file:
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@@
-	)
-	(no_connect
-		(at 129.54 102.87)
 	)
 	(no_connect
@@
 	)
 	(no_connect
-		(at 129.54 105.41)
+		(at 101.6 49.53)
+	)
+	(no_connect
+		(at 83.82 95.25)
+	)
+	(no_connect
+		(at 83.82 87.63)
 	)
 	(no_connect
@@
 	(wire
 		(pts
-			(xy 106.68 45.72) (xy 106.68 49.53)
+			(xy 106.68 46.99) (xy 106.68 49.53)
 		)
 		(stroke
@@
 		)
 	)
+	(hierarchical_label "EL_IN1"
+		(shape input)
+		(at 129.54 102.87 0)
+		(effects
+			(font
+				(size 1.27 1.27)
+			)
+			(justify left)
+		)
+	)
 	(hierarchical_label "UHF_SCLK"
 		(shape input)
@@
 		)
 	)
-	(hierarchical_label "UHF_GPIO3"
-		(shape input)
-		(at 83.82 87.63 180)
-		(effects
-			(font
-				(size 1.27 1.27)
-			)
-			(justify right)
+	(hierarchical_label "EL_IN2"
+		(shape input)
+		(at 129.54 105.41 0)
+		(effects
+			(font
+				(size 1.27 1.27)
+			)
+			(justify left)
+		)
+	)
+	(hierarchical_label "EL_ENC_B"
+		(shape input)
+		(at 129.54 90.17 0)
+		(effects
+			(font
+				(size 1.27 1.27)
+			)
+			(justify left)
 		)
 	)
@@
 		)
 	)
-	(hierarchical_label "VHF_GPIO0"
-		(shape input)
-		(at 129.54 90.17 0)
-		(effects
-			(font
-				(size 1.27 1.27)
-			)
-			(justify left)
-		)
-	)
 	(hierarchical_label "UHF_MOSI"
 		(shape input)
@@
 		)
 	)
-	(hierarchical_label "VHF_GPIO2"
+	(hierarchical_label "VHF_CSN"
+		(shape input)
+		(at 129.54 77.47 0)
+		(effects
+			(font
+				(size 1.27 1.27)
+			)
+			(justify left)
+		)
+	)
+	(hierarchical_label "EL_ENC_A"
 		(shape input)
 		(at 129.54 87.63 0)
@@
 		)
 	)
-	(hierarchical_label "VHF_CSN"
-		(shape input)
-		(at 129.54 77.47 0)
-		(effects
-			(font
-				(size 1.27 1.27)
-			)
-			(justify left)
-		)
-	)
 	(hierarchical_label "UHF_GPIO0"
 		(shape input)
@@
 		)
 	)
-	(hierarchical_label "UHF_GPIO2"
-		(shape input)
-		(at 83.82 95.25 180)
-		(effects
-			(font
-				(size 1.27 1.27)
-			)
-			(justify right)
-		)
-	)
 	(hierarchical_label "VHF_SCLK"
 		(shape input)
@@
 		)
 	)
-	(hierarchical_label "VHF_GPIO3"
+	(hierarchical_label "IMU_CS"
 		(shape input)
 		(at 129.54 100.33 0)
@@
 	(symbol
 		(lib_id "power:+5V")
-		(at 106.68 45.72 0)
+		(at 106.68 46.99 0)
 		(unit 1)
 		(body_style 1)
@@
 		(fields_autoplaced yes)
 		(property "Reference" "#PWR038"
-			(at 106.68 49.53 0)
+			(at 106.68 50.8 0)
 			(hide yes)
 			(show_name no)
@@
 		)
 		(property "Value" "+5V_USB"
-			(at 106.68 40.64 0)
+			(at 106.68 41.91 0)
 			(show_name no)
 			(do_not_autoplace no)
@@
 		)
 		(property "Footprint" ""
-			(at 106.68 45.72 0)
+			(at 106.68 46.99 0)
 			(hide yes)
 			(show_name no)
@@
 		)
 		(property "Datasheet" ""
-			(at 106.68 45.72 0)
+			(at 106.68 46.99 0)
 			(hide yes)
 			(show_name no)
@@
 		)
 		(property "Description" "Power symbol creates a global label with name \"+5V\""
-			(at 106.68 45.72 0)
+			(at 106.68 46.99 0)
 			(hide yes)
 			(show_name no)
@@
 					(unit 1)
 				)
-			)
-		)
-	)
-	(symbol
-		(lib_id "power:+5V")
-		(at 101.6 49.53 0)
-		(unit 1)
-		(body_style 1)
-		(exclude_from_sim no)
-		(in_bom yes)
-		(on_board yes)
-		(in_pos_files yes)
-		(dnp no)
-		(fields_autoplaced yes)
-		(property "Reference" "#PWR037"
-			(at 101.6 53.34 0)
-			(hide yes)
-			(show_name no)
-			(do_not_autoplace no)
-			(effects
-				(font
-					(size 1.27 1.27)
-				)
-			)
-		)
-		(property "Value" "+5V"
-			(at 101.6 44.45 0)
-			(show_name no)
-			(do_not_autoplace no)
-			(effects
-				(font
-					(size 1.27 1.27)
-				)
-			)
-		)
-		(property "Footprint" ""
-			(at 101.6 49.53 0)
-			(hide yes)
-			(show_name no)
-			(do_not_autoplace no)
-			(effects
-				(font
-					(size 1.27 1.27)
-				)
-			)
-		)
-		(property "Datasheet" ""
-			(at 101.6 49.53 0)
-			(hide yes)
-			(show_name no)
-			(do_not_autoplace no)
-			(effects
-				(font
-					(size 1.27 1.27)
-				)
-			)
-		)
-		(property "Description" "Power symbol creates a global label with name \"+5V\""
-			(at 101.6 49.53 0)
-			(hide yes)
-			(show_name no)
-			(do_not_autoplace no)
-			(effects
-				(font
-					(size 1.27 1.27)
-				)
-			)
-		)
-		(pin "1"
-		)
-		(instances
-			(project "MOTOR_RF_HAT"
-				(path "/300cf3d4-e317-44c8-acd8-5f9989779c7c/3e644d4e-3c70-4dba-b47a-c0e6db07080d"
-					(reference "#PWR037")
-					(unit 1)
-				)

Commit message: MOTOR_RF_HAT: BOM enrichment + design review fixes + firmware scaffold
BOM enrichment:
- Added LCSC, MPN, and Farnell properties to 122 of 131 components
  across all schematic sheets (remaining 9 are mechanical/test fixtures)
- Sourced all passives (0603 caps/resistors/inductors), ICs (CC1200,
  A4950E, LMR51420, BSS138, WS2812B), connectors (JST-XH, XT30, SMA)

Design review fixes:
- C1 (4.7uF 50V): 0805→1206 (physically impossible in 0805)
- R1/R2: fixed footprint library from Capacitor_SMD to Resistor_SMD

Firmware scaffold (Firmware/rp2040-motor-rf-hat/):
- Complete merged firmware: RF HAT base + rotator motor control
- motor_pwm.cpp refactored for 2-pin A4950 (IN1/IN2, no PWM pin)
- adxl345.cpp with SPI0 mode switching (mode 3 for IMU, mode 0 for VHF)
- proto.c extended with motor messages 0x60-0x69 (SET_POSITION, PARK,
  STOP, HOME, GET_STATUS, SET_GAINS, ZERO, IMU_READ, RECAL)
- Builds clean: 5.7% RAM, 4.2% flash
- Output: motor_rf_hat_firmware.uf2

Co-Authored-By: Claude Opus 4.6 (1M context) <noreply@anthropic.com>
Parts:
- U4: LCSC (none) -> C7203002; MPN (none) -> SC0915
Changed lines of the file:
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@@
 			)
+		)
+		(property "LCSC" "C7203002"
+			(at 0 0 0)
+			(hide yes)
+			(show_name no)
+			(do_not_autoplace no)
+			(effects (font (size 1.27 1.27)))
+		)
+		(property "MPN" "SC0915"
+			(at 0 0 0)
+			(hide yes)
+			(show_name no)
+			(do_not_autoplace no)
+			(effects (font (size 1.27 1.27)))
+		)
+		(property "Farnell" "3643332"
+			(at 0 0 0)
+			(hide yes)
+			(show_name no)
+			(do_not_autoplace no)
+			(effects (font (size 1.27 1.27)))
 		)
 		(pin "30"
